File: HW/TWIST_tester.sch (KiCad schematic (older format))
At the start: 28 parts, among them J1 DB25_MALE, J10 morsett_1x02_MALE, J11 morsett_1x02_MALE, J2 ALIM_JACK, J3 morsett_1x02_MALE, J4 CONN_01X06, J5 morsett_1x02_MALE, J6 CONN_01X04_MALE, J9 morsett_1x03_MALE, T1 TestPoint, T2 TestPoint, T3 TestPoint, T4 TestPoint, T5 TestPoint, T6 TestPoint

Commit message: Add files via upload
Other:
- note added: "Auxiliar channel contactor\n"
- note added: "Relays contactor"
- note added: "Shunt resistor contactor\n"
- note added: "connector to LM35CA temeperature sensor"
- note removed: "Collegamento sensore\n temperatura"
- note removed: "Shunt resistor's terminal contactor\n"
- moved on the sheet: C7, J4, J9, R5
Changed lines of the file:
@@
 L R R5
 U 1 1 59173373
-P 8850 1700
-F 0 "R5" V 8930 1700 50  0000 C CNN
-F 1 "100K" V 8750 1700 50  0000 C CNN
-F 2 "MYLIB:0805" V 8780 1700 50  0001 C CNN
-F 3 "" H 8850 1700 50  0001 C CNN
-	1    8850 1700
+P 9000 2000
+F 0 "R5" V 9080 2000 50  0000 C CNN
+F 1 "100K" V 8900 2000 50  0000 C CNN
+F 2 "MYLIB:0805" V 8930 2000 50  0001 C CNN
+F 3 "" H 9000 2000 50  0001 C CNN
+	1    9000 2000
 	1    0    0    -1
 $EndComp
@@
 L -5V #PWR25
 U 1 1 5917353A
-P 8850 1950
-F 0 "#PWR25" H 8850 2050 50  0001 C CNN
-F 1 "-5V" H 8850 2100 50  0000 C CNN
-F 2 "" H 8850 1950 50  0001 C CNN
-F 3 "" H 8850 1950 50  0001 C CNN
-	1    8850 1950
+P 9000 2250
+F 0 "#PWR25" H 9000 2350 50  0001 C CNN
+F 1 "-5V" H 9000 2400 50  0000 C CNN
+F 2 "" H 9000 2250 50  0001 C CNN
+F 3 "" H 9000 2250 50  0001 C CNN
+	1    9000 2250
 	-1   0    0    1
 $EndComp
@@
 L C C7
 U 1 1 5917662D
-P 9150 950
-F 0 "C7" H 9175 1050 50  0000 L CNN
-F 1 "100nf" H 9175 850 50  0000 L CNN
-F 2 "MYLIB:0805" H 9188 800 50  0001 C CNN
-F 3 "" H 9150 950 50  0001 C CNN
-	1    9150 950
-	1    0    0    -1
-$EndComp
-Text Notes 9150 3450 0    60   ~ 0
+P 9300 1250
+F 0 "C7" H 9325 1350 50  0000 L CNN
+F 1 "100nf" H 9325 1150 50  0000 L CNN
+F 2 "MYLIB:0805" H 9338 1100 50  0001 C CNN
+F 3 "" H 9300 1250 50  0001 C CNN
+	1    9300 1250
+	1    0    0    -1
+$EndComp
+Text Notes 9150 2700 0    60   ~ 0
 Cell connection\n
-Text Notes 9300 2100 0    60   ~ 0
-Collegamento sensore\n temperatura
-Text Notes 9300 4600 0    60   ~ 0
-Shunt resistor's terminal contactor\n
+Text Notes 8350 750  0    60   ~ 0
+connector to LM35CA temeperature sensor
+Text Notes 9000 3950 0    60   ~ 0
+Shunt resistor contactor\n
 Text Label 2250 2700 0    60   ~ 0
 VBATT+
@@
 L +5V #PWR01
 U 1 1 591C3AB9
-P 9500 750
-F 0 "#PWR01" H 9500 600 50  0001 C CNN
-F 1 "+5V" H 9500 890 50  0000 C CNN
-F 2 "" H 9500 750 50  0001 C CNN
-F 3 "" H 9500 750 50  0001 C CNN
-	1    9500 750
+P 9650 1050
+F 0 "#PWR01" H 9650 900 50  0001 C CNN
+F 1 "+5V" H 9650 1190 50  0000 C CNN
+F 2 "" H 9650 1050 50  0001 C CNN
+F 3 "" H 9650 1050 50  0001 C CNN
+	1    9650 1050
 	1    0    0    -1
 $EndComp
@@
 Text Label 4650 3400 2    60   ~ 0
 VBATT+
-Text Label 8750 1450 2    60   ~ 0
+Text Label 8900 1750 2    60   ~ 0
 TEMP
 $Comp
@@
 L morsett_1x03_MALE J9
 U 1 1 591DDC79
-P 9950 1350
-F 0 "J9" H 9950 1525 50  0000 C CNN
-F 1 "morsett_1x03_MALE" H 9950 950 50  0000 C CNN
-F 2 "MYLIB:morsett_1x03" H 9950 1450 50  0001 C CNN
-F 3 "" H 9950 1450 50  0001 C CNN
-	1    9950 1350
+P 10100 1650
+F 0 "J9" H 10100 1825 50  0000 C CNN
+F 1 "morsett_1x03_MALE" H 10100 1250 50  0000 C CNN
+F 2 "MYLIB:morsett_1x03" H 10100 1750 50  0001 C CNN
+F 3 "" H 10100 1750 50  0001 C CNN
+	1    10100 1650
 	-1   0    0    -1
 $EndComp
@@
 Text Label 2100 3500 0    60   ~ 0
 CHK_RE2
-Text Label 5100 6450 1    60   ~ 0
+Text Label 5350 6800 1    60   ~ 0
 CH2
 $Comp
@@
 L GNDA #PWR013
 U 1 1 5967699F
-P 9050 1700
-F 0 "#PWR013" H 9050 1450 50  0001 C CNN
-F 1 "GNDA" H 9050 1550 50  0000 C CNN
-F 2 "" H 9050 1700 50  0001 C CNN
-F 3 "" H 9050 1700 50  0001 C CNN
-	1    9050 1700
+P 9200 2000
+F 0 "#PWR013" H 9200 1750 50  0001 C CNN
+F 1 "GNDA" H 9200 1850 50  0000 C CNN
+F 2 "" H 9200 2000 50  0001 C CNN
+F 3 "" H 9200 2000 50  0001 C CNN
+	1    9200 2000
 	1    0    0    -1
 $EndComp
@@
 L GNDA #PWR014
 U 1 1 59676FD4
-P 9150 1200
-F 0 "#PWR014" H 9150 950 50  0001 C CNN
-F 1 "GNDA" H 9150 1050 50  0000 C CNN
-F 2 "" H 9150 1200 50  0001 C CNN
-F 3 "" H 9150 1200 50  0001 C CNN
-	1    9150 1200
+P 9300 1500
+F 0 "#PWR014" H 9300 1250 50  0001 C CNN
+F 1 "GNDA" H 9300 1350 50  0000 C CNN
+F 2 "" H 9300 1500 50  0001 C CNN
+F 3 "" H 9300 1500 50  0001 C CNN
+	1    9300 1500
 	1    0    0    -1
 $EndComp
@@
 	4900 3400 4650 3400
 Wire Wire Line
-	9650 1650 9050 1650
-Wire Wire Line
-	9050 1650 9050 1700
-Wire Wire Line
-	8850 1450 8850 1550
-Connection ~ 8850 1450
-Wire Wire Line
-	9500 1250 9650 1250
-Wire Wire Line
-	8750 1450 9650 1450
-Wire Wire Line
-	8850 1850 8850 1950
+	9800 1950 9200 1950
+Wire Wire Line
+	9200 1950 9200 2000
+Wire Wire Line
+	9000 1750 9000 1850
+Connection ~ 9000 1750
+Wire Wire Line
+	9650 1550 9800 1550
+Wire Wire Line
+	8900 1750 9800 1750
+Wire Wire Line
+	9000 2150 9000 2250
 Wire Wire Line
 	1300 4600 3700 4600
@@
 	3500 5000 3500 5150
 Wire Wire Line
-	9500 800  9150 800
-Wire Wire Line
-	9150 1100 9150 1200
-Connection ~ 9500 800
+	9650 1100 9300 1100
+Wire Wire Line
+	9300 1400 9300 1500
+Connection ~ 9650 1100
 Wire Wire Line
 	8800 3050 9700 3050
@@
 Connection ~ 9150 3050
 Wire Wire Line
-	9500 750  9500 1250
+	9650 1050 9650 1550
 Wire Wire Line
 	1900 2700 1900 3100
@@
 Wire Wire Line
 	2200 3800 3000 3800
-Text Label 5000 6450 1    60   ~ 0
+Text Label 5250 6800 1    60   ~ 0
 CH7
-Text Label 4700 6625 1    60   ~ 0
+Text Label 4950 6975 1    60   ~ 0
 DPIN4
-Text Label 4800 6625 1    60   ~ 0
+Text Label 5050 6975 1    60   ~ 0
 DPIN2
 Wire Wire Line
@@
 L CONN_01X06 J4
 U 1 1 5A15DD86
-P 4850 7000
-F 0 "J4" H 4850 7350 50  0000 C CNN
-F 1 "CONN_01X06" V 4950 7000 50  0000 C CNN
-F 2 "MYLIB:morsett_1x06_CB" H 4850 7000 50  0001 C CNN
-F 3 "" H 4850 7000 50  0001 C CNN
-	1    4850 7000
+P 5100 7350
+F 0 "J4" H 5100 7700 50  0000 C CNN
+F 1 "CONN_01X06" V 5200 7350 50  0000 C CNN
+F 2 "MYLIB:morsett_1x06_CB" H 5100 7350 50  0001 C CNN
+F 3 "" H 5100 7350 50  0001 C CNN
+	1    5100 7350
 	0    -1   1    0
 $EndComp
@@
 L GNDD #PWR031
 U 1 1 5A163217
-P 4500 6675
-F 0 "#PWR031" H 4500 6425 50  0001 C CNN
-F 1 "GNDD" H 4500 6525 50  0000 C CNN
-F 2 "" H 4500 6675 50  0001 C CNN
-F 3 "" H 4500 6675 50  0001 C CNN
-	1    4500 6675
+P 4750 7025
+F 0 "#PWR031" H 4750 6775 50  0001 C CNN
+F 1 "GNDD" H 4750 6875 50  0000 C CNN
+F 2 "" H 4750 7025 50  0001 C CNN
+F 3 "" H 4750 7025 50  0001 C CNN
+	1    4750 7025
 	0    1    1    0
 $EndComp
@@
 L GNDA #PWR032
 U 1 1 5A163738
-P 4900 6650
-F 0 "#PWR032" H 4900 6400 50  0001 C CNN
-F 1 "GNDA" H 4900 6500 50  0000 C CNN
-F 2 "" H 4900 6650 50  0001 C CNN
-F 3 "" H 4900 6650 50  0001 C CNN
-	1    4900 6650
+P 5150 7000
+F 0 "#PWR032" H 5150 6750 50  0001 C CNN
+F 1 "GNDA" H 5150 6850 50  0000 C CNN
+F 2 "" H 5150 7000 50  0001 C CNN
+F 3 "" H 5150 7000 50  0001 C CNN
+	1    5150 7000
 	-1   0    0    1
 $EndComp
@@
 $EndComp
 Wire Wire Line
-	5000 6450 5000 6800
-Wire Wire Line
-	5100 6450 5100 6800
-Wire Wire Line
-	4900 6650 4900 6800
-Wire Wire Line
-	4600 6675 4600 6800
-Wire Wire Line
-	4600 6675 4500 6675
-Wire Wire Line
-	4700 6625 4700 6800
-Wire Wire Line
-	4800 6625 4800 6800
+	5250 6800 5250 7150
+Wire Wire Line
+	5350 6800 5350 7150
+Wire Wire Line
+	5150 7000 5150 7150
+Wire Wire Line
+	4850 7025 4850 7150
+Wire Wire Line
+	4850 7025 4750 7025
+Wire Wire Line
+	4950 6975 4950 7150
+Wire Wire Line
+	5050 6975 5050 7150
+Text Notes 9150 4800 0    60   ~ 0
+Relays contactor
+Text Notes 4550 6500 0    60   ~ 0
+Auxiliar channel contactor\n
 $EndSCHEMATC
